File: Xbeetrans.brd (EAGLE design)
At the start: 49 x 57 mm, 16 parts, among them IC1 7805T, IC2 7805T, J1 DCJ0202, K1 JS-M1-9V-4

Commit message: Revert "MYSTMARMZ"
This reverts commit 574e46aa263eab85cf76c740bb46a0becdb3f195.
Parts:
- moved LED1 31.5 mm to (59.7, 68.6), turned to 0 degrees
Routing:
- removed copper zone on layer 1, net GND
- removed copper zone on layer 16, net GND
Changed lines of the file:
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@@
 <setting verticaltext="up"/>
 </settings>
-<grid distance="19.685039" unitdist="mil" unit="mil" style="lines" multiple="1" display="yes" altdistance="0.025" altunitdist="inch" altunit="inch"/>
+<grid distance="0.5" unitdist="mm" unit="mm" style="lines" multiple="1" display="yes" altdistance="0.025" altunitdist="inch" altunit="inch"/>
 <layers>
 <layer number="1" name="Top" color="4" fill="1" visible="yes" active="yes"/>
@@
 <element name="IC1" library="adafruit" package="TO220H" value="7805T" x="58.42" y="21.59"/>
 <element name="IC2" library="adafruit" package="TO220H" value="7805T" x="41.91" y="21.59"/>
-<element name="LED1" library="adafruit" package="LED3MM" value="" x="31.42" y="54.69" rot="R90"/>
+<element name="LED1" library="adafruit" package="LED3MM" value="" x="59.69" y="68.58"/>
 <element name="R1" library="rcl" package="0204/5" value="330" x="36.83" y="62.23"/>
 <element name="C3" library="rcl" package="C025-025X050" value="1uF" x="50.8" y="49.53"/>
@@
 <wire x1="38.1" y1="34.29" x2="38.1" y2="49.53" width="0.254" layer="16"/>
 <wire x1="33.48" y1="30.71" x2="38.1" y2="34.29" width="0.254" layer="16"/>
-<polygon width="0.254" layer="16" isolate="0.3048" orphans="yes">
-<vertex x="19.5" y="68"/>
-<vertex x="68.5" y="68"/>
-<vertex x="68.5" y="11"/>
-<vertex x="19.5" y="11"/>
-</polygon>
-<polygon width="0.254" layer="1" isolate="0.3048" orphans="yes">
-<vertex x="19.5" y="68"/>
-<vertex x="68.5" y="68"/>
-<vertex x="68.5" y="11"/>
-<vertex x="19.5" y="11"/>
-</polygon>
+<wire x1="41.91" y1="11.43" x2="58.42" y2="11.43" width="0" layer="19" extent="1-1"/>
+<wire x1="59.69" y1="29.21" x2="58.42" y2="11.43" width="0" layer="19" extent="16-16"/>
 </signal>
 <signal name="N$3">
@@
 <contactref element="LED1" pad="K"/>
 <contactref element="R1" pad="1"/>
-<wire x1="31.42" y1="55.96" x2="34.29" y2="62.23" width="0" layer="19" extent="1-1"/>
+<wire x1="34.29" y1="62.23" x2="60.96" y2="68.58" width="0" layer="19" extent="1-1"/>
 </signal>
 <signal name="N$8">
@@
 <wire x1="26.67" y1="63.5" x2="27.94" y2="64.77" width="0.254" layer="16"/>
 <wire x1="26.67" y1="63.5" x2="26.67" y2="62.865" width="0.254" layer="16"/>
-<wire x1="31.42" y1="53.42" x2="26.67" y2="62.865" width="0" layer="19" extent="1-1"/>
+<wire x1="55.88" y1="64.77" x2="58.42" y2="68.58" width="0" layer="19" extent="16-16"/>
 <wire x1="44.45" y1="11.43" x2="52.07" y2="49.53" width="0" layer="19" extent="1-1"/>
 </signal>
